Commit message: add some new line in urdf and md

File: my_robot.urdf (robot description, URDF)
Before this commit: robot my_robot, 1 links, 0 joints
Links:
- added link lidar; visual cylinder length=0.05 radius=0.1
Joints:
- added joint base_lider_joint: type fixed, parent base_link, child lidar, origin xyz=0 0 0.225 rpy=0 0 0

Commit message: modify code snipped

File: my_robot.urdf (robot description, URDF)
Before this commit: robot my_robot, 2 links, 1 joints
Links:
- added link base_footprint
- added link caster_wheel; visual sphere radius=0.05
- added link left_wheel; visual cylinder length=0.05 radius=0.1
- added link right_wheel; visual cylinder length=0.05 radius=0.1
Joints:
- removed joint base_lider_joint
- added joint base_caster_wheel_joint: type fixed, parent base_link, child caster_wheel, origin xyz=0.2 0 -0.05 rpy=0 0 0
- added joint base_joint: type fixed, parent base_footprint, child base_link, origin xyz=0 0 0.1 rpy=0 0 0
- added joint base_left_wheel_joint: type continuous, parent base_link, child left_wheel, origin xyz=-0.15 0.225 0 rpy=0 0 0, axis 0 1 0
- added joint base_lidar_joint: type fixed, parent base_link, child lidar, origin xyz=0 0 0.225 rpy=0 0 0
- added joint base_right_wheel_joint: type continuous, parent base_link, child right_wheel, origin xyz=-0.15 -0.225 0 rpy=0 0 0, axis 0 1 0

Commit message: modify my urdf code

File: my_robot.urdf (robot description, URDF)
Before this commit: robot my_robot, 6 links, 5 joints
Links:
- removed link left_wheel
- removed link right_wheel
- added link left_back_wheel; visual cylinder length=0.05 radius=0.1
- added link right_back_wheel; visual cylinder length=0.05 radius=0.1
Joints:
- removed joint base_left_wheel_joint
- removed joint base_right_wheel_joint
- added joint base_left_back_wheel_joint: type continuous, parent base_link, child left_back_wheel, origin xyz=-0.15 0.225 0 rpy=0 0 0, axis 0 1 0
- added joint base_right_back_wheel_joint: type continuous, parent base_link, child right_back_wheel, origin xyz=-0.15 -0.225 0 rpy=0 0 0, axis 0 1 0
